File: horny_dom/horny_dom.kicad_pcb (KiCad board)
At the start: 2 copper layers, 19.3 x 60.9 mm, 28 parts, among them J1 USB_C_Receptacle, SW1 SW_Push, U1 MCP73831-2-OT, U3 ASSR-1218

Commit message: upgrade to kicad6
Other:
- net class Default removed
